Commit message: update urdf(toe radius and position) and toe collision detection

File: robot_simulation/laikago_urdf/laikago.urdf (robot description, URDF)
Before this commit: robot plane, 17 links, 16 joints
Links:
- link toeFL: geometry collision sphere radius=0.03; visual sphere radius=0.03
- link toeFR: geometry collision sphere radius=0.03; visual sphere radius=0.03
- link toeRL: geometry collision sphere radius=0.03; visual sphere radius=0.03
- link toeRR: geometry collision sphere radius=0.03; visual sphere radius=0.03
Joints:
- joint jtoeFL: origin xyz=0 0 -0.24 -> xyz=-0.005 0 -0.255
- joint jtoeFR: origin xyz=0 0 -0.24 -> xyz=-0.005 0 -0.255
- joint jtoeRL: origin xyz=0 0 -0.24 -> xyz=-0.005 0 -0.255
- joint jtoeRR: origin xyz=0 0 -0.24 -> xyz=-0.005 0 -0.255

Commit message: update urdf: toe attributes

File: robot_simulation/laikago_urdf/laikago.urdf (robot description, URDF)
Before this commit: robot plane, 17 links, 16 joints
Links:
- link toeFL: mass 0.1 -> 0.001; geometry collision sphere radius=0.03; visual sphere radius=0.0
- link toeFR: mass 0.1 -> 0.001; geometry collision sphere radius=0.03; visual sphere radius=0.0
- link toeRL: mass 0.1 -> 0.001; geometry collision sphere radius=0.03; visual sphere radius=0.0
- link toeRR: mass 0.1 -> 0.001; geometry collision sphere radius=0.03; visual sphere radius=0.0
